File: matrix.sch (KiCad schematic (older format))
At the start: 166 parts, among them SW10 MX, SW11 MX, SW12 MX, SW13 MX, SW14 MX, SW15 MX, SW16 MX, SW17 MX, SW18 MX, SW19 MX, SW2 MX, SW20 MX, SW21 MX, SW22 MX, SW23 MX, SW24 MX, SW25 MX, SW26 MX, SW27 MX, SW28 MX, SW29 MX, SW3 MX, SW30 MX, SW31 MX, SW32 MX, SW33 MX, SW34 MX, SW35 MX, SW36 MX, SW37 MX, SW38 MX, SW39 MX, SW4 MX, SW40 MX, SW41 MX, SW42 MX, SW43 MX, SW44 MX, SW45 MX, SW46 MX, SW47 MX, SW48 MX, SW49 MX, SW5 MX, SW50 MX, SW51 MX, SW52 MX, SW53 MX, SW54 MX, SW55 MX, SW56 MX, SW57 MX, SW58 MX, SW59 MX, SW6 MX, SW60 MX, SW61 MX, SW62 MX, SW63 MX, SW64 MX, SW65 MX, SW66 MX, SW67 MX, SW68 MX, SW69 MX, SW7 MX, SW70 MX, SW71 MX, SW72 MX, SW73 MX, SW74 MX, SW75 MX, SW76 MX, SW77 MX, SW78 MX, SW79 MX, SW8 MX, SW80 MX, SW81 MX, SW82 MX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

Commit message: Add files via upload
updated files, and added pictures of PCB and key layouts
Parts:
- SW17: renamed from SW18; footprint tastatur:SW_Cherry_MX_1.00u_PCB-NO-LED -> Button_Switch_Keyboard:SW_Cherry_MX_1.50u_PCB
- SW18: renamed from SW19; footprint tastatur:SW_Cherry_MX_1.00u_PCB-NO-LED -> Button_Switch_Keyboard:SW_Cherry_MX_1.00u_PCB
- SW29: renamed from SW30; footprint tastatur:SW_Cherry_MX_1.00u_PCB-NO-LED -> Button_Switch_Keyboard:SW_Cherry_MX_1.50u_PCB
- SW30: renamed from SW31; footprint tastatur:SW_Cherry_MX_1.00u_PCB-NO-LED -> Button_Switch_Keyboard:SW_Cherry_MX_1.00u_PCB
- SW33: renamed from SW34; footprint tastatur:SW_Cherry_MX_1.00u_PCB-NO-LED -> Button_Switch_Keyboard:SW_Cherry_MX_1.50u_PCB
- SW34: renamed from SW35; footprint tastatur:SW_Cherry_MX_1.00u_PCB-NO-LED -> Button_Switch_Keyboard:SW_Cherry_MX_1.00u_PCB
- SW72: renamed from SW73; footprint tastatur:SW_Cherry_MX_1.00u_PCB-NO-LED -> Button_Switch_Keyboard:SW_Cherry_MX_1.75u_PCB
- SW73: renamed from SW74; footprint tastatur:SW_Cherry_MX_1.00u_PCB-NO-LED -> Button_Switch_Keyboard:SW_Cherry_MX_1.50u_PCB
- SW74: renamed from SW75; footprint tastatur:SW_Cherry_MX_1.00u_PCB-NO-LED -> Button_Switch_Keyboard:SW_Cherry_MX_1.50u_PCB
- SW75: renamed from SW76; footprint tastatur:SW_Cherry_MX_1.00u_PCB-NO-LED -> Button_Switch_Keyboard:SW_Cherry_MX_1.00u_PCB
- SW77: renamed from SW78; footprint tastatur:SW_Cherry_MX_1.00u_PCB-NO-LED -> Button_Switch_Keyboard:SW_Cherry_MX_6.25u_PCB
- SW78: renamed from SW79; footprint tastatur:SW_Cherry_MX_1.00u_PCB-NO-LED -> Button_Switch_Keyboard:SW_Cherry_MX_1.00u_PCB
- SW80: renamed from SW81; footprint tastatur:SW_Cherry_MX_1.00u_PCB-NO-LED -> Button_Switch_Keyboard:SW_Cherry_MX_1.50u_PCB
- SW81: renamed from SW82; footprint tastatur:SW_Cherry_MX_1.00u_PCB-NO-LED -> Button_Switch_Keyboard:SW_Cherry_MX_1.00u_PCB
- renumbered SW2 to SW1, SW11 to SW10, SW12 to SW11, SW13 to SW12, SW14 to SW13, SW15 to SW14, SW16 to SW15, SW17 to SW16, SW20 to SW19, SW3 to SW2, SW21 to SW20, SW22 to SW21, SW23 to SW22, SW24 to SW23, SW25 to SW24, SW26 to SW25, SW27 to SW26, SW28 to SW27, SW29 to SW28, SW4 to SW3, SW32 to SW31, SW33 to SW32, SW36 to SW35, SW37 to SW36, SW38 to SW37, SW39 to SW38, SW40 to SW39, SW5 to SW4, SW41 to SW40, SW42 to SW41, SW43 to SW42, SW44 to SW43, SW45 to SW44, SW46 to SW45, SW47 to SW46, SW48 to SW47, SW49 to SW48, SW50 to SW49, SW6 to SW5, SW51 to SW50, SW52 to SW51, SW53 to SW52, SW54 to SW53, SW55 to SW54, SW56 to SW55, SW57 to SW56, SW58 to SW57, SW59 to SW58, SW60 to SW59, SW7 to SW6, SW61 to SW60, SW62 to SW61, SW63 to SW62, SW64 to SW63, SW65 to SW64, SW66 to SW65, SW67 to SW66, SW68 to SW67, SW69 to SW68, SW70 to SW69, SW8 to SW7, SW71 to SW70, SW72 to SW71, SW77 to SW76, SW80 to SW79, SW9 to SW8, SW83 to SW82, SW84 to SW83, SW10 to SW9

Commit message: Add files via upload
updated files.
Parts:
- SW17, SW29, SW33, SW74, SW80: value MX -> SW_Cherry_MX_1.50u_PCB
- SW73: footprint Button_Switch_Keyboard:SW_Cherry_MX_1.50u_PCB -> Button_Switch_Keyboard:SW_Cherry_MX_1.00u_PCB
- SW77: value MX -> SW_Cherry_MX_6.26u_PCB
Changed lines of the file:
@@
 P 1350 3050
 F 0 "SW17" V 1350 3228 50  0000 L CNN
-F 1 "MX" H 1350 2750 60  0001 C CNN
+F 1 "SW_Cherry_MX_1.50u_PCB" H 1350 2750 60  0001 C CNN
 F 2 "Button_Switch_Keyboard:SW_Cherry_MX_1.50u_PCB" H 1350 3050 60  0001 C CNN
 F 3 "" H 1350 3050 60  0001 C CNN
@@
 P 11900 3050
 F 0 "SW29" V 11900 3228 50  0000 L CNN
-F 1 "MX" H 11900 2750 60  0001 C CNN
+F 1 "SW_Cherry_MX_1.50u_PCB" H 11900 2750 60  0001 C CNN
 F 2 "Button_Switch_Keyboard:SW_Cherry_MX_1.50u_PCB" H 11900 3050 60  0001 C CNN
 F 3 "" H 11900 3050 60  0001 C CNN
@@
 P 1350 4500
 F 0 "SW33" V 1350 4678 50  0000 L CNN
-F 1 "MX" H 1350 4200 60  0001 C CNN
+F 1 "SW_Cherry_MX_1.50u_PCB" H 1350 4200 60  0001 C CNN
 F 2 "Button_Switch_Keyboard:SW_Cherry_MX_1.50u_PCB" H 1350 4500 60  0001 C CNN
 F 3 "" H 1350 4500 60  0001 C CNN
@@
 F 0 "SW73" V 11850 8328 50  0000 L CNN
 F 1 "MX" H 11850 7850 60  0001 C CNN
-F 2 "Button_Switch_Keyboard:SW_Cherry_MX_1.50u_PCB" H 11850 8150 60  0001 C CNN
+F 2 "Button_Switch_Keyboard:SW_Cherry_MX_1.00u_PCB" H 11850 8150 60  0001 C CNN
 F 3 "" H 11850 8150 60  0001 C CNN
 	1    11850 8150
@@
 P 1300 9850
 F 0 "SW74" V 1300 10028 50  0000 L CNN
-F 1 "MX" H 1300 9550 60  0001 C CNN
+F 1 "SW_Cherry_MX_1.50u_PCB" H 1300 9550 60  0001 C CNN
 F 2 "Button_Switch_Keyboard:SW_Cherry_MX_1.50u_PCB" H 1300 9850 60  0001 C CNN
 F 3 "" H 1300 9850 60  0001 C CNN
@@
 P 3900 9850
 F 0 "SW77" V 3900 10028 50  0000 L CNN
-F 1 "MX" H 3900 9550 60  0001 C CNN
+F 1 "SW_Cherry_MX_6.26u_PCB" H 3900 9550 60  0001 C CNN
 F 2 "Button_Switch_Keyboard:SW_Cherry_MX_6.25u_PCB" H 3900 9850 60  0001 C CNN
 F 3 "" H 3900 9850 60  0001 C CNN
@@
 P 6500 9850
 F 0 "SW80" V 6500 10028 50  0000 L CNN
-F 1 "MX" H 6500 9550 60  0001 C CNN
+F 1 "SW_Cherry_MX_1.50u_PCB" H 6500 9550 60  0001 C CNN
 F 2 "Button_Switch_Keyboard:SW_Cherry_MX_1.50u_PCB" H 6500 9850 60  0001 C CNN
 F 3 "" H 6500 9850 60  0001 C CNN
