File: Keyboard-ISO-diod.kicad_pcb (KiCad board)
At the start: 2 copper layers, 377.5 x 154 mm, 185 parts, among them J1 USB_B_Mini, SW1 SW_PUSH, SW10 MX, SW11 MX, SW12 MX, SW13 MX, SW14 MX, SW15 MX, SW16 MX, SW17 MX, SW18 MX, SW19 MX, SW2 MX, SW20 MX, SW21 MX, SW22 MX, SW23 MX, SW24 MX, SW25 MX, SW26 MX, SW27 MX, SW28 MX, SW29 MX, SW3 MX, SW30 MX, SW31 MX, SW32 MX, SW33 MX, SW34 MX, SW35 MX, SW36 MX, SW37 MX, SW38 MX, SW39 MX, SW4 MX, SW40 MX, SW41 MX, SW42 MX, SW43 MX, SW44 MX, SW45 MX, SW46 MX, SW47 MX, SW48 MX, SW49 MX, SW5 MX, SW50 MX, SW51 MX, SW52 MX, SW53 MX, SW54 MX, SW55 MX, SW56 MX, SW57 MX, SW58 MX, SW59 MX, SW6 MX, SW60 MX, SW61 MX, SW62 MX, SW63 MX, SW64 MX, SW65 MX, SW66 MX, SW67 MX, SW68 MX, SW69 MX, SW7 MX, SW70 MX, SW71 MX, SW72 MX, SW73 MX, SW74 MX, SW75 MX, SW76 MX, SW77 MX, SW78 MX, SW79 MX, SW8 MX, SW80 MX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

Commit message: updated files
Updated files, changed to using a Teensy++2.0 that plugs right in to the board
Parts:
- removed C1, C2, C3, C4: 0.1uF, Capacitor_SMD:CP_Elec_3x5.3
- removed C5: 4.7uF, Capacitor_SMD:CP_Elec_3x5.3
- removed C6: 1uF, Capacitor_SMD:CP_Elec_3x5.3
- removed C7, C8: 22pF, Capacitor_SMD:CP_Elec_3x5.3
- removed J1: USB_B_Mini, Connector_USB:USB_Micro-B_Amphenol_10103594-0001LF_Horizontal
- removed R4: 10k, Resistor_SMD:R_0603_1608Metric_Pad1.05x0.95mm_HandSolder
- removed the SW1 at (523.0, 174.0)
- removed the SW19 at (70.5, 105.5)
- removed the SW31 at (341.0, 105.5)
- removed the SW35 at (80.0, 129.5)
- removed the SW76 at (77.0, 197.4)
- removed the SW79 at (253.5, 197.5)
- removed the SW82 at (341.0, 187.9)
- removed X1: XTAL_GND, Button_Switch_Keyboard:Crystal_SMD_3225-4pin_3.2x2.5mm
- added J2: Conn_01x01_Female, MountingHole:MountingHole_4.5mm_Pad, F.Cu at (395.0, 68.5)
- added J3: Conn_01x01_Female, MountingHole:MountingHole_4.5mm_Pad, F.Cu at (32.5, 68.5)
- added J4: Conn_01x01_Female, MountingHole:MountingHole_4.5mm_Pad, F.Cu at (395.0, 216.5)
- added J5: Conn_01x01_Female, MountingHole:MountingHole_4.5mm_Pad, F.Cu at (32.5, 216.5)
- added SW17: SW_Cherry_MX_1.50u_PCB, Button_Switch_Keyboard:SW_Cherry_MX_1.50u_PCB, F.Cu at (56.0, 105.5)
- added SW29: SW_Cherry_MX_1.50u_PCB, Button_Switch_Keyboard:SW_Cherry_MX_1.50u_PCB, F.Cu at (305.0, 105.4)
- added SW33: SW_Cherry_MX_1.50u_PCB, Button_Switch_Keyboard:SW_Cherry_MX_1.50u_PCB, F.Cu at (55.0, 129.4)
- added SW72: MX, Button_Switch_Keyboard:SW_Cherry_MX_1.75u_PCB, F.Cu at (302.0, 175.5)
- added SW77: SW_Cherry_MX_6.26u_PCB, Button_Switch_Keyboard:SW_Cherry_MX_6.25u_PCB, F.Cu at (189.0, 198.4)
- added SW80: SW_Cherry_MX_1.50u_PCB, Button_Switch_Keyboard:SW_Cherry_MX_1.50u_PCB, F.Cu at (304.5, 198.4)
- D1, D2, D3: value LED -> LTL-4233
- R1, R2: value 22 -> 330; footprint Resistor_SMD:R_0603_1608Metric_Pad1.05x0.95mm_HandSolder -> Resistor_THT:R_Axial_DIN0204_L3.6mm_D1.6mm_P5.08mm_Horizontal
- R3: value 10K -> 330; footprint Resistor_SMD:R_0603_1608Metric_Pad1.05x0.95mm_HandSolder -> Resistor_THT:R_Axial_DIN0204_L3.6mm_D1.6mm_P5.08mm_Horizontal
- SW18, SW30, SW34, SW73, SW75, SW78, SW81: footprint tastatur:SW_Cherry_MX_1.00u_PCB-NO-LED -> Button_Switch_Keyboard:SW_Cherry_MX_1.00u_PCB
- SW74: value MX -> SW_Cherry_MX_1.50u_PCB; footprint tastatur:SW_Cherry_MX_1.00u_PCB-NO-LED -> Button_Switch_Keyboard:SW_Cherry_MX_1.50u_PCB
- U1: value ATMEGA32U4 -> Teensy++2.0_(Arduino); footprint Button_Switch_Keyboard:ATMEGA32U4-AU -> Teensy:Teensy2.0-pins-headers
- moved D33 375.8 mm to (335.4, 123.0)
- moved D36 371.8 mm to (51.0, 146.5)
- moved D34 365.2 mm to (354.4, 123.0)
- moved D37 353.8 mm to (74.0, 146.5)
- moved D76 349.0 mm to (335.5, 186.5)
- moved D86 348.3 mm to (374.4, 191.5)
- moved D38 348.2 mm to (94.0, 146.5)
- moved D32 340.6 mm to (298.9, 122.0)
- moved D53 333.0 mm to (79.0, 169.5)
- moved D85 326.8 mm to (354.5, 191.5)
- moved D54 321.1 mm to (98.0, 169.5)
- moved D31 311.2 mm to (268.9, 122.5)
- moved D84 310.9 mm to (335.0, 191.5)
- moved D81 305.2 mm to (252.5, 215.5)
- moved D44 303.8 mm to (213.0, 146.5)
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- renumbered SW2 to SW1, SW11 to SW10, SW12 to SW11, SW13 to SW12, SW14 to SW13, SW15 to SW14, SW16 to SW15, SW17 to SW16, SW20 to SW19, SW3 to SW2, SW21 to SW20, SW22 to SW21, SW23 to SW22, SW24 to SW23, SW25 to SW24, SW26 to SW25, SW27 to SW26, SW28 to SW27, SW29 to SW28, SW4 to SW3, SW32 to SW31, SW33 to SW32, SW36 to SW35, SW37 to SW36, SW38 to SW37, SW39 to SW38, SW40 to SW39, SW5 to SW4, SW41 to SW40, SW42 to SW41, SW43 to SW42, SW44 to SW43, SW45 to SW44, SW46 to SW45, SW47 to SW46, SW48 to SW47, SW49 to SW48, SW50 to SW49, SW6 to SW5, SW51 to SW50, SW52 to SW51, SW53 to SW52, SW54 to SW53, SW55 to SW54, SW56 to SW55, SW57 to SW56, SW58 to SW57, SW59 to SW58, SW60 to SW59, SW7 to SW6, SW61 to SW60, SW62 to SW61, SW63 to SW62, SW64 to SW63, SW65 to SW64, SW66 to SW65, SW67 to SW66, SW68 to SW67, SW69 to SW68, SW70 to SW69, SW8 to SW7, SW71 to SW70, SW72 to SW71, SW77 to SW76, SW80 to SW79, SW9 to SW8, SW83 to SW82, SW84 to SW83, SW10 to SW9
Connections:
- D1 pad 1: +5V -> GND
- D1 pad 2: /capslock -> Net-(D1-Pad2)
- D2 pad 1: +5V -> GND
- D2 pad 2: /scroll-lock -> Net-(D2-Pad2)
- D3 pad 1: +5V -> GND
- D3 pad 2: /QWERTY-DVORAK -> Net-(D3-Pad2)
- R1 pad 1: Net-(R1-Pad1) -> Net-(D1-Pad2)
- R1 pad 2: Net-(J1-Pad3) -> Net-(R1-Pad2)
- R2 pad 1: Net-(R2-Pad1) -> Net-(D2-Pad2)
- R2 pad 2: Net-(J1-Pad2) -> Net-(R2-Pad2)
- R3 pad 1: Net-(R3-Pad1) -> Net-(D3-Pad2)
- R3 pad 2: VCC -> Net-(R3-Pad2)
- SW18 pad 2: Net-(D20-Pad2) -> Net-(D21-Pad2)
- SW30 pad 2: Net-(D32-Pad2) -> Net-(D33-Pad2)
- SW34 pad 2: Net-(D36-Pad2) -> Net-(D37-Pad2)
- SW73 pad 2: Net-(D75-Pad2) -> Net-(D76-Pad2)
- SW74 pad 1: ROW5 -> ROW6
- SW74 pad 2: Net-(D76-Pad2) -> Net-(D77-Pad2)
- SW75 pad 2: Net-(D77-Pad2) -> Net-(D78-Pad2)
- SW78 pad 2: Net-(D80-Pad2) -> Net-(D81-Pad2)
- SW81 pad 2: Net-(D83-Pad2) -> Net-(D84-Pad2)
- U1 pad 1: Net-(U1-Pad1) -> GND
- U1 pad 10: COL13 -> COL8
- U1 pad 11: COL14 -> COL7
- U1 pad 12: COL15 -> COL6
- U1 pad 13: Net-(R3-Pad1) -> COL15
- U1 pad 14: VCC -> COL16
- U1 pad 15: GND -> COL13
- U1 pad 16: Net-(C7-Pad1) -> COL14
- U1 pad 17: Net-(C8-Pad1) -> Net-(R1-Pad2)
- U1 pad 18: /capslock -> Net-(R2-Pad2)
- U1 pad 19: /scroll-lock -> Net-(R3-Pad2)
- U1 pad 2: VCC -> (no net)
- U1 pad 20: /QWERTY-DVORAK -> COL12
- U1 pad 21: Net-(U1-Pad21) -> (no net)
- U1 pad 22: Net-(U1-Pad22) -> GND
- U1 pad 23: GND -> (no net)
- U1 pad 24: VCC -> COL11
- U1 pad 25: COL10 -> COL5
- U1 pad 26: COL9 -> ROW6
- U1 pad 27: COL8 -> ROW5
- U1 pad 28: COL7 -> ROW4
- U1 pad 29: COL6 -> ROW3
- U1 pad 3: Net-(R2-Pad1) -> (no net)
- U1 pad 30: COL5 -> ROW2
- U1 pad 31: COL4 -> ROW1
- U1 pad 32: COL3 -> (no net)
- U1 pad 33: Net-(R4-Pad2) -> GND
- U1 pad 34: VCC -> (no net)
- U1 pad 35: GND -> COL1
- U1 pad 37: COL1 -> COL3
- U1 pad 38: ROW6 -> COL4
- U1 pad 39: ROW4 -> (no net)
- U1 pad 4: Net-(R1-Pad1) -> (no net)
- U1 pad 40: ROW3 -> (no net)
- U1 pad 41: ROW2 -> (no net)
- U1 pad 42: ROW1 -> (no net)
- U1 pad 43: GND -> (no net)
- U1 pad 5: GND -> (no net)
- U1 pad 6: Net-(C6-Pad1) -> (no net)
- U1 pad 7: VCC -> COL10
- U1 pad 8: COL11 -> COL9
- U1 pad 9: COL12 -> (no net)
Other:
- board size 377.5 x 154 mm -> 377 x 162.5 mm
- board text added: "QWE/ DVOR"
- board text added: "caps lock"
- board text added: "scroll lock"
