File: Keyboard-ISO.kicad_pcb (KiCad board)
At the start: 2 copper layers, 400 x 154 mm, 174 parts, among them J1 DB25_Female, J2 Conn_01x01_Female, J3 Conn_01x01_Female, J4 Conn_01x01_Female, J5 Conn_01x01_Female, SW10 MX, SW11 MX, SW12 MX, SW13 MX, SW14 MX, SW15 MX, SW16 MX, SW17 MX, SW18 MX, SW19 MX, SW2 MX, SW20 MX, SW21 MX, SW22 MX, SW23 MX, SW24 MX, SW25 MX, SW26 MX, SW27 MX, SW28 MX, SW29 MX, SW3 MX, SW30 MX, SW31 MX, SW32 MX, SW33 MX, SW34 MX, SW35 MX, SW36 MX, SW37 MX, SW38 MX, SW39 MX, SW4 MX, SW40 MX, SW41 MX, SW42 MX, SW43 MX, SW44 MX, SW45 MX, SW46 MX, SW47 MX, SW48 MX, SW49 MX, SW5 MX, SW50 MX, SW51 MX, SW52 MX, SW53 MX, SW54 MX, SW55 MX, SW56 MX, SW57 MX, SW58 MX, SW59 MX, SW6 MX, SW60 MX, SW61 MX, SW62 MX, SW63 MX, SW64 MX, SW65 MX, SW66 MX, SW67 MX, SW68 MX, SW69 MX, SW7 MX, SW70 MX, SW71 MX, SW72 MX, SW73 MX, SW74 MX, SW75 MX, SW76 MX, SW77 MX, SW78 MX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

Commit message: Add files via upload
updated files, and added pictures of PCB and key layouts
Parts:
- removed the SW19 at (70.5, 105.5)
- removed the SW31 at (341.0, 105.5)
- removed the SW35 at (80.0, 129.5)
- removed the SW76 at (77.0, 198.4)
- removed the SW79 at (253.5, 197.5)
- removed the SW82 at (341.0, 198.0)
- added SW17: MX, Button_Switch_Keyboard:SW_Cherry_MX_1.50u_PCB, F.Cu at (56.0, 105.5)
- added SW29: MX, Button_Switch_Keyboard:SW_Cherry_MX_1.50u_PCB, F.Cu at (305.0, 105.4)
- added SW33: MX, Button_Switch_Keyboard:SW_Cherry_MX_1.50u_PCB, F.Cu at (55.0, 129.4)
- added SW72: MX, Button_Switch_Keyboard:SW_Cherry_MX_1.75u_PCB, F.Cu at (302.0, 175.5)
- added SW77: MX, Button_Switch_Keyboard:SW_Cherry_MX_6.25u_PCB, F.Cu at (189.0, 198.4)
- added SW80: MX, Button_Switch_Keyboard:SW_Cherry_MX_1.50u_PCB, F.Cu at (304.5, 198.4)
- SW18, SW30, SW34, SW75, SW78, SW81: footprint tastatur:SW_Cherry_MX_1.00u_PCB-NO-LED -> Button_Switch_Keyboard:SW_Cherry_MX_1.00u_PCB
- SW73, SW74: footprint tastatur:SW_Cherry_MX_1.00u_PCB-NO-LED -> Button_Switch_Keyboard:SW_Cherry_MX_1.50u_PCB
- moved SW74 287.4 mm to (74.5, 198.4)
- moved SW78 85.5 mm to (259.0, 198.4)
- moved SW73 58.5 mm to (361.0, 175.4)
- moved SW75 42.0 mm to (99.0, 198.4)
- moved SW81 38.5 mm to (341.0, 198.0)
- moved D78 37.3 mm to (92.5, 215.5)
- moved SW30 33.0 mm to (341.0, 106.0)
- moved SW18 30.0 mm to (80.5, 105.5)
- moved D80 29.9 mm to (182.9, 215.5), turned to 0 degrees
- moved D77 29.4 mm to (67.9, 215.5), turned to 0 degrees
- moved SW34 23.0 mm to (80.0, 129.5)
- moved SW76 22.0 mm to (119.0, 198.4)
- moved D48 21.2 mm to (301.4, 165.0)
- moved SW61 18.5 mm to (75.0, 175.4)
- moved D64 18.5 mm to (67.5, 191.5)
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- renumbered J4 to J2, J2 to J3, J5 to J4, J3 to J5, SW2 to SW1, SW11 to SW10, SW12 to SW11, SW13 to SW12, SW14 to SW13, SW15 to SW14, SW16 to SW15, SW17 to SW16, SW20 to SW19, SW3 to SW2, SW21 to SW20, SW22 to SW21, SW23 to SW22, SW24 to SW23, SW25 to SW24, SW26 to SW25, SW27 to SW26, SW28 to SW27, SW29 to SW28, SW4 to SW3, SW32 to SW31, SW33 to SW32, SW36 to SW35, SW37 to SW36, SW38 to SW37, SW39 to SW38, SW40 to SW39, SW5 to SW4, SW41 to SW40, SW42 to SW41, SW43 to SW42, SW44 to SW43, SW45 to SW44, SW46 to SW45, SW47 to SW46, SW48 to SW47, SW49 to SW48, SW50 to SW49, SW6 to SW5, SW51 to SW50, SW52 to SW51, SW53 to SW52, SW54 to SW53, SW55 to SW54, SW56 to SW55, SW57 to SW56, SW58 to SW57, SW59 to SW58, SW60 to SW59, SW7 to SW6, SW61 to SW60, SW62 to SW61, SW63 to SW62, SW64 to SW63, SW65 to SW64, SW66 to SW65, SW67 to SW66, SW68 to SW67, SW69 to SW68, SW70 to SW69, SW8 to SW7, SW71 to SW70, SW72 to SW71, SW77 to SW76, SW80 to SW79, SW9 to SW8, SW83 to SW82, SW84 to SW83, SW10 to SW9
Connections:
- SW18 pad 2: Net-(D20-Pad2) -> Net-(D21-Pad2)
- SW30 pad 2: Net-(D32-Pad2) -> Net-(D33-Pad2)
- SW34 pad 2: Net-(D36-Pad2) -> Net-(D37-Pad2)
- SW73 pad 2: Net-(D75-Pad2) -> Net-(D76-Pad2)
- SW74 pad 1: ROW5 -> ROW6
- SW74 pad 2: Net-(D76-Pad2) -> Net-(D77-Pad2)
- SW75 pad 2: Net-(D77-Pad2) -> Net-(D78-Pad2)
- SW78 pad 2: Net-(D80-Pad2) -> Net-(D81-Pad2)
- SW81 pad 2: Net-(D83-Pad2) -> Net-(D84-Pad2)
Routing:
- net /GND: track 662.0 -> 684.0 mm
- net ROW5: track 382.6 -> 364.6 mm
- net Net-(D48-Pad2): track 13.0 -> 26.9 mm
- net COL9: track 342.4 -> 329.2 mm
- net COL1: track 474.3 -> 487.3 mm
- net COL4: track 450.1 -> 437.3 mm
- net COL10: track 339.6 -> 329.0 mm
- net COL2: track 467.5 -> 477.5 mm
- net COL3: track 447.5 -> 456.9 mm
- net Net-(D81-Pad2): track 8.67 -> 17.6 mm
- net Net-(D82-Pad2): track 9.58 -> 17.8 mm
- net Net-(D78-Pad2): track 9.85 -> 17.6 mm
- net COL8: track 353.9 -> 346.3 mm
- net ROW4: track 368.5 -> 360.9 mm
- net Net-(D80-Pad2): track 10.3 -> 17.8 mm
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- added copper zone on B.Cu, net /GND
- removed copper zone on F.Cu, net (none)
Other:
- board size 400 x 154 mm -> 400 x 162.5 mm

Commit message: Add files via upload
updated files.
Parts:
- SW17, SW33, SW74, SW80: value MX -> SW_Cherry_MX_1.50u_PCB
- SW73: footprint Button_Switch_Keyboard:SW_Cherry_MX_1.50u_PCB -> Button_Switch_Keyboard:SW_Cherry_MX_1.00u_PCB
- SW77: value MX -> SW_Cherry_MX_6.26u_PCB
- moved J1 19.1 mm to (398.4, 151.1)
- moved D76 12.3 mm to (355.5, 169.0), turned to 0 degrees
- moved D85 0.88 mm to (354.5, 191.5)
Routing:
- net ROW5: track 364.6 -> 339.0 mm, vias 0 -> 1
- net ROW6: track 397.0 -> 374.6 mm
- net ROW4: track 360.9 -> 339.9 mm
- net COL14: track 133.3 -> 113.0 mm
- net COL3: track 456.9 -> 437.0 mm
- net COL5: track 416.4 -> 396.5 mm
- net COL2: track 477.5 -> 457.7 mm
- net COL16: track 92.9 -> 73.6 mm
- net COL6: track 404.6 -> 385.4 mm
- net COL13: track 222.3 -> 203.2 mm
- net COL4: track 437.3 -> 418.4 mm
- net COL11: track 270.7 -> 252.0 mm
- net COL12: track 248.9 -> 230.2 mm
- net COL15: track 115.7 -> 97.4 mm
- net ROW2: track 400.5 -> 383.2 mm
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- removed copper zone on B.Cu, net /GND
Other:
- board size 400 x 162.5 mm -> 385 x 162.5 mm

Commit message: updated files
Updated files, changed to using a Teensy++2.0 that plugs right in to the board
Parts:
- removed J1: DB25_Female, Connector_Dsub:DSUB-25_Female_Vertical_P2.77x2.84mm_MountingHoles
- added R1: 330, Resistor_THT:R_Axial_DIN0204_L3.6mm_D1.6mm_P5.08mm_Horizontal, F.Cu at (313.5, 67.0)
- added R2: 330, Resistor_THT:R_Axial_DIN0204_L3.6mm_D1.6mm_P5.08mm_Horizontal, F.Cu at (317.5, 67.0)
- added R3: 330, Resistor_THT:R_Axial_DIN0204_L3.6mm_D1.6mm_P5.08mm_Horizontal, F.Cu at (321.0, 67.0)
- added U1: Teensy++2.0_(Arduino), Teensy:Teensy2.0-pins-headers, F.Cu at (376.5, 161.0)
- D1, D2, D3: value LED -> LTL-4233
- SW29: value MX -> SW_Cherry_MX_1.50u_PCB
- moved D76 26.6 mm to (335.5, 186.5)
Connections:
- net /GND renamed GND
Routing:
- net Net-(R1-Pad2): track 0.00 -> 107.8 mm
- net Net-(R2-Pad2): track 0.00 -> 101.3 mm
- net Net-(R3-Pad2): track 0.00 -> 95.3 mm
- net COL7: track 398.0 -> 345.1 mm
- net COL5: track 396.5 -> 346.1 mm
- net GND: track 667.9 -> 716.0 mm
- net Net-(D1-Pad2): track 78.5 -> 31.0 mm
- net ROW5: track 339.0 -> 293.3 mm, vias 1 -> 0
- net COL13: track 203.2 -> 161.6 mm
- net COL11: track 252.0 -> 210.7 mm
- net ROW4: track 339.9 -> 304.5 mm
- net COL12: track 230.2 -> 196.8 mm
- net ROW6: track 374.6 -> 342.9 mm
- net COL14: track 113.0 -> 83.2 mm
- net COL9: track 319.7 -> 290.7 mm
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- added copper zone on B.Cu, net GND
Other:
- board size 385 x 162.5 mm -> 377 x 162.5 mm
- board text added: "*"
